File: RAC-altimeter.sch (EAGLE design)
At the start: 0 parts

Commit message: Added altimeter and MCU
Parts:
- added IC1: MAX32660GWE+, MAX32660GWE+:MAX32660GWE+
- added IC2: BMP388, BMP388:BMP388
- added Y1: 32.768kHz, ST2012SB32768B0HPWB4:ST2012SB32768B0HPWB4
Connections:
- new net N$1: IC1.32KOUT, Y1.2
- new net N$2: IC1.32KIN, Y1.1
- new net SPI0_MISO: IC1.P0.4
- new net SPI0_MOSI: IC1.P0.5
- new net SPI0_SCK: IC1.P0.6
