File: RAC-altimeter.sch (EAGLE design)
At the start: 14 parts, among them IC2 BMP388, IC3 STM32L412KBU6, J1 MICRO-SD

Commit message: Connected the BMI088 IMU, removed pull-up on SD data line
Parts:
- removed R4: 10k, SparkFun-Resistors:10KOHM-0603-1/10W-1%
- added C3, C4: 0.1uF, SparkFun-Capacitors:0.1UF-0603-25V-(+80/-20%)
- added IC1: BMI088, BMI088:BMI088
Connections:
- net GND: now also C3.2, C4.1, IC1.GNDA, IC1.GNDIO, IC1.SDO1, IC1.SDO2
- net I2C1_SCL: now also IC1.SCL/SCK
- net I2C1_SDA: now also IC1.SDA/SDI
- net SPI1_MISO: no longer R4.1
- net VCC: now also C3.1, C4.2, IC1.PS, IC1.VDD, IC1.VDDIO; no longer R4.2
Changed lines of the file:
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@@
 <part name="SUPPLY3" library="SparkFun-PowerSymbols" library_urn="urn:adsk.eagle:library:530" deviceset="VCC" device=""/>
 <part name="GND4" library="SparkFun-PowerSymbols" library_urn="urn:adsk.eagle:library:530" deviceset="GND" device=""/>
-<part name="R4" library="SparkFun-Resistors" library_urn="urn:adsk.eagle:library:532" deviceset="10KOHM" device="-0603-1/10W-1%" package3d_urn="urn:adsk.eagle:package:39650/1" value="10k"/>
 <part name="IC3" library="STM32L412KBU6" deviceset="STM32L412KBU6" device=""/>
 <part name="C6" library="SparkFun-Capacitors" deviceset="0.1UF" device="-0603-25V-(+80/-20%)" value="0.1uF"/>
@@
 <part name="R7" library="SparkFun-Resistors" deviceset="4.7KOHM" device="-0603-1/10W-1%" value="4.7k"/>
 <part name="SUPPLY7" library="SparkFun-PowerSymbols" library_urn="urn:adsk.eagle:library:530" deviceset="VCC" device=""/>
+<part name="IC1" library="BMI088" deviceset="BMI088" device=""/>
+<part name="SUPPLY1" library="SparkFun-PowerSymbols" library_urn="urn:adsk.eagle:library:530" deviceset="VCC" device=""/>
+<part name="SUPPLY4" library="SparkFun-PowerSymbols" library_urn="urn:adsk.eagle:library:530" deviceset="VCC" device=""/>
+<part name="GND2" library="SparkFun-PowerSymbols" library_urn="urn:adsk.eagle:library:530" deviceset="GND" device=""/>
+<part name="C3" library="SparkFun-Capacitors" deviceset="0.1UF" device="-0603-25V-(+80/-20%)" value="0.1uF"/>
+<part name="C4" library="SparkFun-Capacitors" deviceset="0.1UF" device="-0603-25V-(+80/-20%)" value="0.1uF"/>
+<part name="GND5" library="SparkFun-PowerSymbols" library_urn="urn:adsk.eagle:library:530" deviceset="GND" device=""/>
 </parts>
 <sheets>
@@
 <attribute name="VALUE" x="154.94" y="17.526" size="1.778" layer="96" align="top-center"/>
 </instance>
-<instance part="SUPPLY2" gate="G$1" x="139.7" y="48.26" smashed="yes">
-<attribute name="VALUE" x="139.7" y="51.054" size="1.778" layer="96" align="bottom-center"/>
+<instance part="SUPPLY2" gate="G$1" x="139.7" y="40.64" smashed="yes">
+<attribute name="VALUE" x="139.7" y="43.434" size="1.778" layer="96" align="bottom-center"/>
 </instance>
 <instance part="GND3" gate="1" x="129.54" y="63.5" smashed="yes">
@@
 <attribute name="VALUE" x="187.96" y="63.246" size="1.778" layer="96" align="top-center"/>
 </instance>
-<instance part="R4" gate="G$1" x="134.62" y="38.1" smashed="yes" rot="R90">
-<attribute name="NAME" x="133.096" y="38.1" size="1.778" layer="95" font="vector" rot="R90" align="bottom-center"/>
-<attribute name="VALUE" x="136.144" y="38.1" size="1.778" layer="96" font="vector" rot="R90" align="top-center"/>
-</instance>
 <instance part="IC3" gate="G$1" x="5.08" y="58.42" smashed="yes">
 <attribute name="NAME" x="46.99" y="81.28" size="1.778" layer="95" align="center-left"/>
@@
 <instance part="SUPPLY7" gate="G$1" x="68.58" y="66.04" smashed="yes">
 <attribute name="VALUE" x="68.58" y="68.834" size="1.778" layer="96" align="bottom-center"/>
+</instance>
+<instance part="IC1" gate="G$1" x="132.08" y="121.92" smashed="yes">
+<attribute name="NAME" x="138.43" y="129.54" size="1.778" layer="95" align="center-left"/>
+<attribute name="VALUE" x="138.43" y="127" size="1.778" layer="96" align="center-left"/>
+</instance>
+<instance part="SUPPLY1" gate="G$1" x="111.76" y="121.92" smashed="yes" rot="MR0">
+<attribute name="VALUE" x="111.76" y="124.714" size="1.778" layer="96" rot="MR0" align="bottom-center"/>
+</instance>
+<instance part="SUPPLY4" gate="G$1" x="193.04" y="121.92" smashed="yes">
+<attribute name="VALUE" x="193.04" y="124.714" size="1.778" layer="96" align="bottom-center"/>
+</instance>
+<instance part="GND2" gate="1" x="127" y="99.06" smashed="yes">
+<attribute name="VALUE" x="127" y="98.806" size="1.778" layer="96" align="top-center"/>
+</instance>
+<instance part="C3" gate="G$1" x="121.92" y="111.76" smashed="yes" rot="MR0">
+<attribute name="NAME" x="120.396" y="114.681" size="1.778" layer="95" font="vector" rot="MR0"/>
+<attribute name="VALUE" x="120.396" y="109.601" size="1.778" layer="96" font="vector" rot="MR0"/>
+</instance>
+<instance part="C4" gate="G$1" x="180.34" y="111.76" smashed="yes" rot="MR180">
+<attribute name="NAME" x="181.864" y="108.839" size="1.778" layer="95" font="vector" rot="MR180"/>
+<attribute name="VALUE" x="181.864" y="113.919" size="1.778" layer="96" font="vector" rot="MR180"/>
+</instance>
+<instance part="GND5" gate="1" x="180.34" y="99.06" smashed="yes">
+<attribute name="VALUE" x="180.34" y="98.806" size="1.778" layer="96" align="top-center"/>
 </instance>
 </instances>
@@
 <segment>
 <pinref part="J1" gate="J1" pin="DO"/>
-<wire x1="160.02" y1="30.48" x2="134.62" y2="30.48" width="0.1524" layer="91"/>
-<label x="129.54" y="30.48" size="1.778" layer="95" rot="MR0"/>
-<pinref part="R4" gate="G$1" pin="1"/>
-<wire x1="134.62" y1="30.48" x2="129.54" y2="30.48" width="0.1524" layer="91"/>
-<wire x1="134.62" y1="30.48" x2="134.62" y2="33.02" width="0.1524" layer="91"/>
-<junction x="134.62" y="30.48"/>
+<wire x1="160.02" y1="30.48" x2="154.94" y2="30.48" width="0.1524" layer="91"/>
+<label x="154.94" y="30.48" size="1.778" layer="95" rot="MR0"/>
 </segment>
 <segment>
@@
 <wire x1="17.78" y1="93.98" x2="17.78" y2="83.82" width="0.1524" layer="91"/>
 </segment>
+<segment>
+<pinref part="IC1" gate="G$1" pin="GNDIO"/>
+<wire x1="132.08" y1="109.22" x2="127" y2="109.22" width="0.1524" layer="91"/>
+<pinref part="GND2" gate="1" pin="GND"/>
+<wire x1="127" y1="109.22" x2="127" y2="101.6" width="0.1524" layer="91"/>
+<pinref part="IC1" gate="G$1" pin="GNDA"/>
+<wire x1="132.08" y1="114.3" x2="127" y2="114.3" width="0.1524" layer="91"/>
+<wire x1="127" y1="114.3" x2="127" y2="109.22" width="0.1524" layer="91"/>
+<junction x="127" y="109.22"/>
+<pinref part="C3" gate="G$1" pin="2"/>
+<wire x1="121.92" y1="109.22" x2="127" y2="109.22" width="0.1524" layer="91"/>
+</segment>
+<segment>
+<pinref part="GND5" gate="1" pin="GND"/>
+<pinref part="C4" gate="G$1" pin="1"/>
+<wire x1="180.34" y1="106.68" x2="180.34" y2="101.6" width="0.1524" layer="91"/>
+<pinref part="IC1" gate="G$1" pin="SDO2"/>
+<wire x1="167.64" y1="119.38" x2="172.72" y2="119.38" width="0.1524" layer="91"/>
+<wire x1="172.72" y1="119.38" x2="172.72" y2="106.68" width="0.1524" layer="91"/>
+<pinref part="IC1" gate="G$1" pin="SDO1"/>
+<wire x1="167.64" y1="106.68" x2="172.72" y2="106.68" width="0.1524" layer="91"/>
+<wire x1="172.72" y1="106.68" x2="180.34" y2="106.68" width="0.1524" layer="91"/>
+<junction x="172.72" y="106.68"/>
+<junction x="180.34" y="106.68"/>
+</segment>
 </net>
 <net name="I2C1_SCL" class="0">
@@
 <junction x="73.66" y="45.72"/>
 </segment>
+<segment>
+<pinref part="IC1" gate="G$1" pin="SCL/SCK"/>
+<wire x1="132.08" y1="104.14" x2="111.76" y2="104.14" width="0.1524" layer="91"/>
+<label x="111.76" y="104.14" size="1.778" layer="95" rot="MR0"/>
+</segment>
 </net>
 <net name="I2C1_SDA" class="0">
@@
 <junction x="63.5" y="48.26"/>
 </segment>
+<segment>
+<pinref part="IC1" gate="G$1" pin="SDA/SDI"/>
+<wire x1="167.64" y1="121.92" x2="172.72" y2="121.92" width="0.1524" layer="91"/>
+<label x="172.72" y="121.92" size="1.778" layer="95"/>
+</segment>
 </net>
 <net name="VCC" class="0">
@@
 <wire x1="160.02" y1="35.56" x2="139.7" y2="35.56" width="0.1524" layer="91"/>
 <pinref part="SUPPLY2" gate="G$1" pin="VCC"/>
-<wire x1="139.7" y1="35.56" x2="139.7" y2="45.72" width="0.1524" layer="91"/>
-<pinref part="R4" gate="G$1" pin="2"/>
-<wire x1="139.7" y1="45.72" x2="139.7" y2="48.26" width="0.1524" layer="91"/>
-<wire x1="134.62" y1="43.18" x2="134.62" y2="45.72" width="0.1524" layer="91"/>
-<wire x1="134.62" y1="45.72" x2="139.7" y2="45.72" width="0.1524" layer="91"/>
-<junction x="139.7" y="45.72"/>
+<wire x1="139.7" y1="35.56" x2="139.7" y2="40.64" width="0.1524" layer="91"/>
 </segment>
 <segment>
@@
 <pinref part="SUPPLY7" gate="G$1" pin="VCC"/>
 </segment>
-</net>
+<segment>
+<pinref part="IC1" gate="G$1" pin="PS"/>
+<wire x1="132.08" y1="106.68" x2="111.76" y2="106.68" width="0.1524" layer="91"/>
+<wire x1="111.76" y1="106.68" x2="111.76" y2="116.84" width="0.1524" layer="91"/>
+<pinref part="SUPPLY1" gate="G$1" pin="VCC"/>
+<pinref part="C3" gate="G$1" pin="1"/>
+<pinref part="IC1" gate="G$1" pin="VDD"/>
+<wire x1="111.76" y1="116.84" x2="111.76" y2="121.92" width="0.1524" layer="91"/>
+<wire x1="121.92" y1="116.84" x2="132.08" y2="116.84" width="0.1524" layer="91"/>
+<wire x1="121.92" y1="116.84" x2="111.76" y2="116.84" width="0.1524" layer="91"/>
+<junction x="121.92" y="116.84"/>
+<junction x="111.76" y="116.84"/>
+</segment>
+<segment>
+<pinref part="IC1" gate="G$1" pin="VDDIO"/>
+<wire x1="167.64" y1="116.84" x2="180.34" y2="116.84" width="0.1524" layer="91"/>
+<wire x1="180.34" y1="116.84" x2="180.34" y2="114.3" width="0.1524" layer="91"/>
+<pinref part="C4" gate="G$1" pin="2"/>
+<wire x1="180.34" y1="116.84" x2="193.04" y2="116.84" width="0.1524" layer="91"/>
+<junction x="180.34" y="116.84"/>
+<pinref part="SUPPLY4" gate="G$1" pin="VCC"/>
+<wire x1="193.04" y1="116.84" x2="193.04" y2="121.92" width="0.1524" layer="91"/>
+</segment>
+</net>
